Commit message: gibbon model files update

File: catkin_ws/src/gibbon/urdf/gibbon.urdf (robot description, URDF)
Before this commit: robot gibbon, 9 links, 8 joints
Links:
- removed link base_link
- added link link_1_tip, mass 1e-05
- added link link_2_tip, mass 1e-05
- link link_1: geometry collision cylinder length=0.7 radius=0.01; visual cylinder length=0.7 radius=0.01
- link link_1_gripper_pole: mass 0.001 -> 1e-05
- link link_2: geometry collision cylinder length=0.7 radius=0.01; visual cylinder length=0.7 radius=0.01
- link link_2_gripper_pole: mass 0.001 -> 1e-05
Joints:
- removed joint base_link__link_1
- added joint link_1__link_1_tip: type revolute, parent link_1, child link_1_tip, origin xyz=0 0 0.1 rpy=0 0 0, limit lower=0 upper=0 effort=0 velocity=0
- added joint link_2__link_2_tip: type revolute, parent link_2, child link_2_tip, origin xyz=0.02 0 0.7999999999999999 rpy=0 0 0, limit lower=0 upper=0 effort=0 velocity=0
- joint link_1__link_2: limit lower=-3.141592653589793 upper=3.141592653589793 effort=0 velocity=0 -> lower=-3.141592653589793 upper=3.141592653589793 effort=10000.0 velocity=10.0; origin xyz=0.01 0 -1 rpy=0 0 0 -> xyz=0.01 0 -0.7 rpy=3.141592653589793 0 0
- joint link_2__gripper: origin xyz=0.02 0 -1 rpy=0 1.5707963267948966 0 -> xyz=0.02 0 0.7 rpy=0 -1.5707963267948966 0
