Commit message: ladder default origin inertia

File: catkin_ws/src/gibbon/urdf/ladder.xacro (robot description, xacro)
@@ -33,134 +33,134 @@
   <link name='ladder__link_0'>
     <inertial>
+      <!-- <origin rpy="1.57 0 0" xyz="0 0.15 3"/> -->
+      <mass value="1.0"/>
+      <inertia ixx="0.1633333333333333" ixy="0.0" ixz="0.0" iyy="0" iyz="0.0" izz="0.0"/>
+    </inertial>
+    <visual>
+      <origin rpy="1.57 0 0" xyz="0 0 3"/>
+      <geometry>
+        <cylinder length="0.3" radius="0.01"/>
+      </geometry>
+    </visual>
+    <visual>
       <origin rpy="1.57 0 0" xyz="0 0.15 3"/>
-      <mass value="1.0"/>
-      <inertia ixx="0.1633333333333333" ixy="0.0" ixz="0.0" iyy="0" iyz="0.0" izz="0.0"/>
-    </inertial>
-    <visual>
+      <geometry>
+        <cylinder length="0.01" radius="0.02"/>
+      </geometry>
+    </visual>
+    <visual>
+      <origin rpy="1.57 0 0" xyz="0 -0.15 3"/>
+      <geometry>
+        <cylinder length="0.01" radius="0.02"/>
+      </geometry>
+    </visual>
+    <collision>
       <origin rpy="1.57 0 0" xyz="0 0 3"/>
       <geometry>
         <cylinder length="0.3" radius="0.01"/>
       </geometry>
-    </visual>
-    <visual>
+    </collision>
+    <collision>
       <origin rpy="1.57 0 0" xyz="0 0.15 3"/>
       <geometry>
         <cylinder length="0.01" radius="0.02"/>
       </geometry>
-    </visual>
-    <visual>
+    </collision>
+    <collision>
       <origin rpy="1.57 0 0" xyz="0 -0.15 3"/>
       <geometry>
         <cylinder length="0.01" radius="0.02"/>
       </geometry>
-    </visual>
-    <collision>
-      <origin rpy="1.57 0 0" xyz="0 0 3"/>
-      <geometry>
-        <cylinder length="0.3" radius="0.01"/>
-      </geometry>
-    </collision>
-    <collision>
-      <origin rpy="1.57 0 0" xyz="0 0.15 3"/>
-      <geometry>
-        <cylinder length="0.01" radius="0.02"/>
-      </geometry>
-    </collision>
-    <collision>
-      <origin rpy="1.57 0 0" xyz="0 -0.15 3"/>
-      <geometry>
-        <cylinder length="0.01" radius="0.02"/>
-      </geometry>
     </collision>
   </link>
   <link name='ladder__link_1'>
     <inertial>
+      <!-- <origin rpy="1.57 0 0" xyz="1.4 0.15 3"/> -->
+      <mass value="1.0"/>
+      <inertia ixx="0.1633333333333333" ixy="0.0" ixz="0.0" iyy="0" iyz="0.0" izz="0.0"/>
+    </inertial>
+    <visual>
+      <origin rpy="1.57 0 0" xyz="1.4 0 3"/>
+      <geometry>
+        <cylinder length="0.3" radius="0.01"/>
+      </geometry>
+    </visual>
+    <visual>
       <origin rpy="1.57 0 0" xyz="1.4 0.15 3"/>
-      <mass value="1.0"/>
-      <inertia ixx="0.1633333333333333" ixy="0.0" ixz="0.0" iyy="0" iyz="0.0" izz="0.0"/>
-    </inertial>
-    <visual>
+      <geometry>
+        <cylinder length="0.01" radius="0.02"/>
+      </geometry>
+    </visual>
+    <visual>
+      <origin rpy="1.57 0 0" xyz="1.4 -0.15 3"/>
+      <geometry>
+        <cylinder length="0.01" radius="0.02"/>
+      </geometry>
+    </visual>
+    <collision>
       <origin rpy="1.57 0 0" xyz="1.4 0 3"/>
       <geometry>
         <cylinder length="0.3" radius="0.01"/>
       </geometry>
-    </visual>
-    <visual>
+    </collision>
+    <collision>
       <origin rpy="1.57 0 0" xyz="1.4 0.15 3"/>
       <geometry>
         <cylinder length="0.01" radius="0.02"/>
       </geometry>
-    </visual>
-    <visual>
+    </collision>
+    <collision>
       <origin rpy="1.57 0 0" xyz="1.4 -0.15 3"/>
       <geometry>
         <cylinder length="0.01" radius="0.02"/>
       </geometry>
-    </visual>
-    <collision>
-      <origin rpy="1.57 0 0" xyz="1.4 0 3"/>
-      <geometry>
-        <cylinder length="0.3" radius="0.01"/>
-      </geometry>
-    </collision>
-    <collision>
-      <origin rpy="1.57 0 0" xyz="1.4 0.15 3"/>
-      <geometry>
-        <cylinder length="0.01" radius="0.02"/>
-      </geometry>
-    </collision>
-    <collision>
-      <origin rpy="1.57 0 0" xyz="1.4 -0.15 3"/>
-      <geometry>
-        <cylinder length="0.01" radius="0.02"/>
-      </geometry>
     </collision>
   </link>
   <link name='ladder__link_2'>
     <inertial>
+      <!-- <origin rpy="1.57 0 0" xyz="2.8 0.15 3"/> -->
+      <mass value="1.0"/>
+      <inertia ixx="0.1633333333333333" ixy="0.0" ixz="0.0" iyy="0" iyz="0.0" izz="0.0"/>
+    </inertial>
+    <visual>
+      <origin rpy="1.57 0 0" xyz="2.8 0 3"/>
+      <geometry>
+        <cylinder length="0.3" radius="0.01"/>
+      </geometry>
+    </visual>
+    <visual>
       <origin rpy="1.57 0 0" xyz="2.8 0.15 3"/>
-      <mass value="1.0"/>
-      <inertia ixx="0.1633333333333333" ixy="0.0" ixz="0.0" iyy="0" iyz="0.0" izz="0.0"/>
-    </inertial>
-    <visual>
+      <geometry>
+        <cylinder length="0.01" radius="0.02"/>
+      </geometry>
+    </visual>
+    <visual>
+      <origin rpy="1.57 0 0" xyz="2.8 -0.15 3"/>
+      <geometry>
+        <cylinder length="0.01" radius="0.02"/>
+      </geometry>
+    </visual>
+    <collision>
       <origin rpy="1.57 0 0" xyz="2.8 0 3"/>
       <geometry>
         <cylinder length="0.3" radius="0.01"/>
       </geometry>
-    </visual>
-    <visual>
+    </collision>
+    <collision>
       <origin rpy="1.57 0 0" xyz="2.8 0.15 3"/>
       <geometry>
         <cylinder length="0.01" radius="0.02"/>
       </geometry>
-    </visual>
-    <visual>
+    </collision>
+    <collision>
       <origin rpy="1.57 0 0" xyz="2.8 -0.15 3"/>
       <geometry>
         <cylinder length="0.01" radius="0.02"/>
       </geometry>
-    </visual>
-    <collision>
-      <origin rpy="1.57 0 0" xyz="2.8 0 3"/>
-      <geometry>
-        <cylinder length="0.3" radius="0.01"/>
-      </geometry>
-    </collision>
-    <collision>
-      <origin rpy="1.57 0 0" xyz="2.8 0.15 3"/>
-      <geometry>
-        <cylinder length="0.01" radius="0.02"/>
-      </geometry>
-    </collision>
-    <collision>
-      <origin rpy="1.57 0 0" xyz="2.8 -0.15 3"/>
-      <geometry>
-        <cylinder length="0.01" radius="0.02"/>
-      </geometry>
     </collision>
   </link>
   <link name='ladder__link_3'>
     <inertial>
-      <origin rpy="1.57 0 0" xyz="4.2 0.15 3"/>
+      <!-- <origin rpy="1.57 0 0" xyz="4.2 0.15 3"/> -->
       <mass value="1.0"/>
       <inertia ixx="0.1633333333333333" ixy="0.0" ixz="0.0" iyy="0" iyz="0.0" izz="0.0"/>
