Commit message: tf go

File: catkin_ws/src/gibbon/urdf/gibbon.xacro (robot description, xacro)
@@ -3,9 +3,7 @@
     <xacro:property name="arm_radius" value="0.02" />
     <xacro:property name="arm_len" value="0.7" />
+    <xacro:property name="PI" value="3.14159265359" />
     <material name="grey1"><color rgba="0.95 0.95 0.95 1"/></material>
     <material name="grey2"><color rgba="0.91 0.91 0.91 1"/></material>
-    <link name='base_link'>
-      <origin rpy="0 0 0" xyz="0 0 0"/>
-    </link>
     <link name='link_1'>
       <origin rpy="0 0 0" xyz="0 0 0"/>
@@ -18,5 +16,5 @@
     </link>
     <link name='link_2'>
-      <origin rpy="0 0 0" xyz="0 0.02 0"/>
+      <origin rpy="${PI/2} 0 0" xyz="0 0.52 0"/>
       <material name="grey1"/>
       <visual name='visual'>
@@ -26,11 +24,9 @@
       </visual>
     </link>
-    <joint name="base_link__link_1" type="fixed">
-      <parent link="base_link"/>
-      <child link="link_1"/>
-    </joint>
-    <joint name="base_link__link_2" type="fixed">
-      <parent link="base_link"/>
+    <joint name="link_1__link_2" type="revolute">
+      <parent link="link_1"/>
       <child link="link_2"/>
+      <limit effort="1000.0" lower="${-PI}" upper="${PI}" velocity="0.5"/>
+      <origin rpy=".5 0 0" xyz="${arm_radius+1} 0 0.2"/>
     </joint>
 </robot>

Commit message: link placement

File: catkin_ws/src/gibbon/urdf/gibbon.xacro (robot description, xacro)
@@ -4,10 +4,11 @@
     <xacro:property name="arm_len" value="0.7" />
     <xacro:property name="PI" value="3.14159265359" />
-    <material name="grey1"><color rgba="0.95 0.95 0.95 1"/></material>
-    <material name="grey2"><color rgba="0.91 0.91 0.91 1"/></material>
+    <material name="grey1"><color rgba="1 1 1 1"/></material>
+    <material name="grey2"><color rgba="0.31 0.31 0.31 1"/></material>
     <link name='link_1'>
       <origin rpy="0 0 0" xyz="0 0 0"/>
-      <material name="grey2"/>
       <visual name='visual'>
+        <origin rpy="0 0 0" xyz="0 0 -${arm_len/2}"/>
+        <material name="grey2"/>
         <geometry>
           <cylinder radius="${arm_radius}" length="${arm_len}"/>
@@ -16,7 +17,8 @@
     </link>
     <link name='link_2'>
-      <origin rpy="${PI/2} 0 0" xyz="0 0.52 0"/>
-      <material name="grey1"/>
+      <origin rpy="0 0 0" xyz="${arm_radius*2} 0 0"/>
       <visual name='visual'>
+        <origin rpy="0 0 0" xyz="${arm_radius*2} 0 -${arm_len/2}"/>
+        <material name="grey1"/>
         <geometry>
           <cylinder radius="${arm_radius}" length="${arm_len}"/>
@@ -24,9 +26,3 @@
       </visual>
     </link>
-    <joint name="link_1__link_2" type="revolute">
-      <parent link="link_1"/>
-      <child link="link_2"/>
-      <limit effort="1000.0" lower="${-PI}" upper="${PI}" velocity="0.5"/>
-      <origin rpy=".5 0 0" xyz="${arm_radius+1} 0 0.2"/>
-    </joint>
 </robot>

Commit message: fix missed joint

File: catkin_ws/src/gibbon/urdf/gibbon.xacro (robot description, xacro)
@@ -26,3 +26,9 @@
       </visual>
     </link>
+    <joint name="link_1__link_2" type="revolute">
+      <parent link="link_1"/>
+      <child link="link_2"/>
+      <limit effort="1000.0" lower="${-PI}" upper="${PI}" velocity="0.5"/>
+      <origin rpy=".5 0 0" xyz="${arm_radius+1} 0 0.2"/>
+    </joint>
 </robot>

Commit message: fixing joint

File: catkin_ws/src/gibbon/urdf/gibbon.xacro (robot description, xacro)
@@ -29,6 +29,6 @@
       <parent link="link_1"/>
       <child link="link_2"/>
-      <limit effort="1000.0" lower="${-PI}" upper="${PI}" velocity="0.5"/>
-      <origin rpy=".5 0 0" xyz="${arm_radius+1} 0 0.2"/>
+      <limit effort="1000.0" lower="${-pi}" upper="${pi}" velocity="0.5"/>
+      <origin rpy="0 0 0" xyz="${arm_radius} 0 -${arm_len}"/>
     </joint>
 </robot>

Commit message: grippers added

File: catkin_ws/src/gibbon/urdf/gibbon.xacro (robot description, xacro)
@@ -3,7 +3,15 @@
     <xacro:property name="arm_radius" value="0.02" />
     <xacro:property name="arm_len" value="0.7" />
-    <xacro:property name="PI" value="3.14159265359" />
+    <!-- <xacro:property name="PI" value="3.14159265359" /> -->
+    <xacro:property name="width" value="0.2" />
+    <xacro:property name="polelen" value="0.0" />
     <material name="grey1"><color rgba="1 1 1 1"/></material>
     <material name="grey2"><color rgba="0.31 0.31 0.31 1"/></material>
+    <xacro:macro name="default_inertial" params="mass">
+      <inertial>
+        <mass value="${mass}" />
+        <inertia ixx="1.0" ixy="0.0" ixz="0.0" iyy="1.0" iyz="0.0" izz="1.0" />
+      </inertial>
+    </xacro:macro>
     <link name='link_1'>
       <origin rpy="0 0 0" xyz="0 0 0"/>
@@ -32,3 +40,90 @@
       <origin rpy="0 0 0" xyz="${arm_radius} 0 -${arm_len}"/>
     </joint>
+    <joint name="link_1__gripper" type="fixed">
+      <parent link="link_1"/>
+      <child link="link_1_gripper_pole"/>
+      <origin rpy="0 -${pi/2} 0" xyz="0 0 0"/>
+    </joint>
+    <joint name="link_2__gripper" type="fixed">
+      <parent link="link_2"/>
+      <child link="link_2_gripper_pole"/>
+      <origin rpy="0 ${pi/2} 0" xyz="${arm_radius*2} 0 -${arm_len}"/>
+    </joint>
+    <link name="link_1_gripper_pole">
+      <visual>
+        <geometry>
+          <cylinder length="${polelen}" radius="0.01"/>
+        </geometry>
+        <origin xyz="0 0 0" rpy="0 0 0 "/>
+      </visual>
+      <collision>
+        <geometry>
+          <cylinder length="${polelen}" radius="0.01"/>
+        </geometry>
+        <origin xyz="0 0 0" rpy="0 0 0 "/>
+      </collision>
+      <xacro:default_inertial mass="0.05"/>
+    </link>
+    <link name="link_2_gripper_pole">
+      <visual>
+        <geometry>
+          <cylinder length="${polelen}" radius="0.01"/>
+        </geometry>
+        <origin xyz="0 0 0" rpy="0 0 0 "/>
+      </visual>
+      <collision>
+        <geometry>
+          <cylinder length="${polelen}" radius="0.01"/>
+        </geometry>
+        <origin xyz="0 0 0" rpy="0 0 0 "/>
+      </collision>
+      <xacro:default_inertial mass="0.05"/>
+    </link>
+    <xacro:macro name="gripper" params="prefix reflect link_name">
+      <joint name="${link_name}_${prefix}_gripper_joint" type="revolute">
+        <axis xyz="0 0 ${reflect}"/>
+        <limit effort="1000.0" lower="0.0" upper="0.548" velocity="0.5"/>
+        <origin rpy="0 0 0" xyz="${polelen} ${reflect*0.01} 0"/>
+        <parent link="${link_name}_gripper_pole"/>
+        <child link="${link_name}_${prefix}_gripper"/>
+      </joint>
+      <link name="${link_name}_${prefix}_gripper">
+        <visual>
+          <origin rpy="${(reflect-1)/2*pi} 0 0" xyz="0 0 0"/>
+          <geometry>
+            <mesh filename="package://urdf_tutorial/meshes/l_finger.dae"/>
+          </geometry>
+        </visual>
+        <collision>
+          <geometry>
+            <mesh filename="package://urdf_tutorial/meshes/l_finger.dae"/>
+          </geometry>
+          <origin rpy="${(reflect-1)/2*pi} 0 0" xyz="0 0 0"/>
+        </collision>
+        <xacro:default_inertial mass="0.05"/>
+      </link>
+      <joint name="${link_name}_${prefix}_tip_joint" type="fixed">
+        <parent link="${link_name}_${prefix}_gripper"/>
+        <child link="${link_name}_${prefix}_tip"/>
+      </joint>
+      <link name="${link_name}_${prefix}_tip">
+        <visual>
+          <origin rpy="${(reflect-1)/2*pi} 0 0" xyz="0.09137 0.00495 0"/>
+          <geometry>
+            <mesh filename="package://urdf_tutorial/meshes/l_finger_tip.dae"/>
+          </geometry>
+        </visual>
+        <collision>
+          <geometry>
+            <mesh filename="package://urdf_tutorial/meshes/l_finger_tip.dae"/>
+          </geometry>
+          <origin rpy="${(reflect-1)/2*pi} 0 0" xyz="0.09137 0.00495 0"/>
+        </collision>
+        <xacro:default_inertial mass="0.05"/>
+      </link>
+    </xacro:macro>
+    <xacro:gripper prefix="left" reflect="1" link_name="link_1" />
+    <xacro:gripper prefix="right" reflect="-1" link_name="link_1" />
+    <xacro:gripper prefix="left" reflect="1" link_name="link_2" />
+    <xacro:gripper prefix="right" reflect="-1" link_name="link_2" />
 </robot>

Commit message: base_link added

File: catkin_ws/src/gibbon/urdf/gibbon.xacro (robot description, xacro)
@@ -3,5 +3,4 @@
     <xacro:property name="arm_radius" value="0.02" />
     <xacro:property name="arm_len" value="0.7" />
-    <!-- <xacro:property name="PI" value="3.14159265359" /> -->
     <xacro:property name="width" value="0.2" />
     <xacro:property name="polelen" value="0.0" />
@@ -14,4 +13,10 @@
       </inertial>
     </xacro:macro>
+    <link name="base_link"/>
+    <joint name="base_link__link_1" type="fixed">
+      <parent link="base_link"/>
+      <child link="link_1"/>
+      <origin rpy="0 0 0" xyz="0 0 0"/>
+    </joint>
     <link name='link_1'>
       <origin rpy="0 0 0" xyz="0 0 0"/>
@@ -23,4 +28,5 @@
         </geometry>
       </visual>
+      <xacro:default_inertial mass="0.5"/>
     </link>
     <link name='link_2'>
@@ -33,4 +39,5 @@
         </geometry>
       </visual>
+      <xacro:default_inertial mass="0.5"/>
     </link>
     <joint name="link_1__link_2" type="revolute">
@@ -63,5 +70,5 @@
         <origin xyz="0 0 0" rpy="0 0 0 "/>
       </collision>
-      <xacro:default_inertial mass="0.05"/>
+      <xacro:default_inertial mass="0.001"/>
     </link>
     <link name="link_2_gripper_pole">
@@ -78,5 +85,5 @@
         <origin xyz="0 0 0" rpy="0 0 0 "/>
       </collision>
-      <xacro:default_inertial mass="0.05"/>
+      <xacro:default_inertial mass="0.001"/>
     </link>
     <xacro:macro name="gripper" params="prefix reflect link_name">

Commit message: collision + inertia

File: catkin_ws/src/gibbon/urdf/gibbon.xacro (robot description, xacro)
@@ -3,4 +3,5 @@
     <xacro:property name="arm_radius" value="0.02" />
     <xacro:property name="arm_len" value="0.7" />
+    <xacro:property name="arm_mass" value="1.0" />
     <xacro:property name="width" value="0.2" />
     <xacro:property name="polelen" value="0.0" />
@@ -11,4 +12,10 @@
         <mass value="${mass}" />
         <inertia ixx="1.0" ixy="0.0" ixz="0.0" iyy="1.0" iyz="0.0" izz="1.0" />
+      </inertial>
+    </xacro:macro>
+    <xacro:macro name="arm_inertial" params="mass len">
+      <inertial>
+        <mass value="${mass}" />
+        <inertia ixx="${1.0 / 3.0 * mass * len * len}" ixy="0.0" ixz="0.0" iyy="${1.0 / 3.0 * mass * len * len}" iyz="0.0" izz="0.0" />
       </inertial>
     </xacro:macro>
@@ -28,5 +35,10 @@
         </geometry>
       </visual>
-      <xacro:default_inertial mass="0.5"/>
+      <collision>
+        <geometry>
+          <cylinder radius="${arm_radius}" length="${arm_len}"/>
+        </geometry>
+      </collision>
+      <xacro:arm_inertial mass="${arm_mass}" len="${arm_len}"/>
     </link>
     <link name='link_2'>
@@ -39,5 +51,10 @@
         </geometry>
       </visual>
-      <xacro:default_inertial mass="0.5"/>
+      <collision>
+        <geometry>
+          <cylinder radius="${arm_radius}" length="${arm_len}"/>
+        </geometry>
+      </collision>
+      <xacro:arm_inertial mass="${arm_mass}" len="${arm_len}"/>
     </link>
     <joint name="link_1__link_2" type="revolute">

Commit message: meshes added

File: catkin_ws/src/gibbon/urdf/gibbon.xacro (robot description, xacro)
@@ -116,10 +116,10 @@
           <origin rpy="${(reflect-1)/2*pi} 0 0" xyz="0 0 0"/>
           <geometry>
-            <mesh filename="package://urdf_tutorial/meshes/l_finger.dae"/>
+            <mesh filename="package://gibbon/meshes/l_finger.dae"/>
           </geometry>
         </visual>
         <collision>
           <geometry>
-            <mesh filename="package://urdf_tutorial/meshes/l_finger.dae"/>
+            <mesh filename="package://gibbon/meshes/l_finger.dae"/>
           </geometry>
           <origin rpy="${(reflect-1)/2*pi} 0 0" xyz="0 0 0"/>
@@ -135,10 +135,10 @@
           <origin rpy="${(reflect-1)/2*pi} 0 0" xyz="0.09137 0.00495 0"/>
           <geometry>
-            <mesh filename="package://urdf_tutorial/meshes/l_finger_tip.dae"/>
+            <mesh filename="package://gibbon/meshes/l_finger_tip.dae"/>
           </geometry>
         </visual>
         <collision>
           <geometry>
-            <mesh filename="package://urdf_tutorial/meshes/l_finger_tip.dae"/>
+            <mesh filename="package://gibbon/meshes/l_finger_tip.dae"/>
           </geometry>
           <origin rpy="${(reflect-1)/2*pi} 0 0" xyz="0.09137 0.00495 0"/>

Commit message: joints publich & control

File: catkin_ws/src/gibbon/urdf/gibbon.xacro (robot description, xacro)
@@ -1,4 +1,4 @@
 <?xml version='1.0'?>
-<robot xmlns:xacro="http://www.ros.org/wiki/xacro" name='monkey'>
+<robot xmlns:xacro="http://www.ros.org/wiki/xacro" name='gibbon'>
     <xacro:property name="arm_radius" value="0.02" />
     <xacro:property name="arm_len" value="0.7" />
@@ -64,4 +64,13 @@
       <origin rpy="0 0 0" xyz="${arm_radius} 0 -${arm_len}"/>
     </joint>
+    <transmission name="link_1__link_2_trans">
+      <type>transmission_interface/SimpleTransmission</type>
+      <actuator name="$link_1__link_2_motor">
+        <mechanicalReduction>1</mechanicalReduction>
+      </actuator>
+      <joint name="link_1__link_2">
+        <hardwareInterface>PositionJointInterface</hardwareInterface>
+      </joint>
+    </transmission>
     <joint name="link_1__gripper" type="fixed">
       <parent link="link_1"/>
@@ -112,4 +121,13 @@
         <child link="${link_name}_${prefix}_gripper"/>
       </joint>
+      <transmission name="${link_name}_${prefix}_gripper_joint_trans">
+        <type>transmission_interface/SimpleTransmission</type>
+        <actuator name="$${link_name}_${prefix}_gripper_joint_motor">
+          <mechanicalReduction>1</mechanicalReduction>
+        </actuator>
+        <joint name="${link_name}_${prefix}_gripper_joint">
+          <hardwareInterface>PositionJointInterface</hardwareInterface>
+        </joint>
+      </transmission>
       <link name="${link_name}_${prefix}_gripper">
         <visual>

Commit message: gripper changed

File: catkin_ws/src/gibbon/urdf/gibbon.xacro (robot description, xacro)
@@ -1,7 +1,7 @@
 <?xml version='1.0'?>
 <robot xmlns:xacro="http://www.ros.org/wiki/xacro" name='gibbon'>
-    <xacro:property name="arm_radius" value="0.02" />
-    <xacro:property name="arm_len" value="0.7" />
-    <xacro:property name="arm_mass" value="1.0" />
+    <xacro:property name="arm_radius" value="0.01" />
+    <xacro:property name="arm_len" value="0.4" />
+    <xacro:property name="arm_mass" value="3.0" />
     <xacro:property name="width" value="0.2" />
     <xacro:property name="polelen" value="0.0" />
@@ -27,5 +27,4 @@
     </joint>
     <link name='link_1'>
-      <origin rpy="0 0 0" xyz="0 0 0"/>
       <visual name='visual'>
         <origin rpy="0 0 0" xyz="0 0 -${arm_len/2}"/>
@@ -36,4 +35,5 @@
       </visual>
       <collision>
+        <origin rpy="0 0 0" xyz="0 0 -${arm_len/2}"/>
         <geometry>
           <cylinder radius="${arm_radius}" length="${arm_len}"/>
@@ -43,5 +43,4 @@
     </link>
     <link name='link_2'>
-      <origin rpy="0 0 0" xyz="${arm_radius*2} 0 0"/>
       <visual name='visual'>
         <origin rpy="0 0 0" xyz="${arm_radius*2} 0 -${arm_len/2}"/>
@@ -52,4 +51,5 @@
       </visual>
       <collision>
+        <origin rpy="0 0 0" xyz="${arm_radius*2} 0 -${arm_len/2}"/>
         <geometry>
           <cylinder radius="${arm_radius}" length="${arm_len}"/>
@@ -132,33 +132,27 @@
       <link name="${link_name}_${prefix}_gripper">
         <visual>
-          <origin rpy="${(reflect-1)/2*pi} 0 0" xyz="0 0 0"/>
+          <origin rpy="${reflect*pi/2} 0 ${reflect*pi/2}" xyz="0.05 0 0"/>
           <geometry>
-            <mesh filename="package://gibbon/meshes/l_finger.dae"/>
+            <box size="0.001 0.02 0.1"/>
           </geometry>
         </visual>
         <collision>
           <geometry>
-            <mesh filename="package://gibbon/meshes/l_finger.dae"/>
+            <box size="0.001 0.02 0.1"/>
           </geometry>
-          <origin rpy="${(reflect-1)/2*pi} 0 0" xyz="0 0 0"/>
+          <origin rpy="${reflect*pi/2} 0 ${reflect*pi/2}" xyz="0.05 0 0"/>
         </collision>
-        <xacro:default_inertial mass="0.05"/>
-      </link>
-      <joint name="${link_name}_${prefix}_tip_joint" type="fixed">
-        <parent link="${link_name}_${prefix}_gripper"/>
-        <child link="${link_name}_${prefix}_tip"/>
-      </joint>
-      <link name="${link_name}_${prefix}_tip">
+        <!-- tips -->
         <visual>
-          <origin rpy="${(reflect-1)/2*pi} 0 0" xyz="0.09137 0.00495 0"/>
+          <origin rpy="0 0 0" xyz="0.1 ${-1*reflect*0.005} 0"/>
           <geometry>
-            <mesh filename="package://gibbon/meshes/l_finger_tip.dae"/>
+            <box size="0.001 0.01 0.02"/>
           </geometry>
         </visual>
         <collision>
           <geometry>
-            <mesh filename="package://gibbon/meshes/l_finger_tip.dae"/>
+            <box size="0.001 0.01 0.02"/>
           </geometry>
-          <origin rpy="${(reflect-1)/2*pi} 0 0" xyz="0.09137 0.00495 0"/>
+          <origin rpy="0 0 0" xyz="0.1 ${-1*reflect*0.005} 0"/>
         </collision>
         <xacro:default_inertial mass="0.05"/>

Commit message: joint limits extented

File: catkin_ws/src/gibbon/urdf/gibbon.xacro (robot description, xacro)
@@ -6,6 +6,6 @@
     <xacro:property name="width" value="0.2" />
     <xacro:property name="polelen" value="0.0" />
-    <material name="grey1"><color rgba="1 1 1 1"/></material>
-    <material name="grey2"><color rgba="0.31 0.31 0.31 1"/></material>
+    <material name="grey1"><color rgba="0.7 0.7 0.7 1"/></material>
+    <material name="grey2"><color rgba="0.9 0.9 0.9 1"/></material>
     <xacro:macro name="default_inertial" params="mass">
       <inertial>
@@ -27,5 +27,5 @@
     </joint>
     <link name='link_1'>
-      <visual name='visual'>
+      <visual>
         <origin rpy="0 0 0" xyz="0 0 -${arm_len/2}"/>
         <material name="grey2"/>
@@ -43,5 +43,5 @@
     </link>
     <link name='link_2'>
-      <visual name='visual'>
+      <visual>
         <origin rpy="0 0 0" xyz="${arm_radius*2} 0 -${arm_len/2}"/>
         <material name="grey1"/>
@@ -61,5 +61,5 @@
       <parent link="link_1"/>
       <child link="link_2"/>
-      <limit effort="1000.0" lower="${-pi}" upper="${pi}" velocity="0.5"/>
+      <limit effort="100000.0" lower="${-pi}" upper="${pi}" velocity="3.14"/>
       <origin rpy="0 0 0" xyz="${arm_radius} 0 -${arm_len}"/>
     </joint>
@@ -117,5 +117,5 @@
       <joint name="${link_name}_${prefix}_gripper_joint" type="revolute">
         <axis xyz="0 0 ${reflect}"/>
-        <limit effort="1000.0" lower="0.0" upper="0.548" velocity="0.5"/>
+        <limit effort="100000.0" lower="0.0" upper="0.548" velocity="3.14"/>
         <origin rpy="0 0 0" xyz="${polelen} ${reflect*0.01} 0"/>
         <parent link="${link_name}_gripper_pole"/>
@@ -145,5 +145,4 @@
           <origin rpy="${reflect*pi/2} 0 ${reflect*pi/2}" xyz="0.05 0 0"/>
         </collision>
-        <!-- tips -->
         <visual>
           <origin rpy="0 0 0" xyz="0.1 ${-1*reflect*0.005} 0"/>

Commit message: Control: solve ode

File: catkin_ws/src/gibbon/urdf/gibbon.xacro (robot description, xacro)
@@ -2,6 +2,6 @@
 <robot xmlns:xacro="http://www.ros.org/wiki/xacro" name='gibbon'>
     <xacro:property name="arm_radius" value="0.01" />
-    <xacro:property name="arm_len" value="0.4" />
-    <xacro:property name="arm_mass" value="3.0" />
+    <xacro:property name="arm_len" value="1" />
+    <xacro:property name="arm_mass" value="1.0" />
     <xacro:property name="width" value="0.2" />
     <xacro:property name="polelen" value="0.0" />

Commit message: main joint dynamics

File: catkin_ws/src/gibbon/urdf/gibbon.xacro (robot description, xacro)
@@ -61,6 +61,8 @@
       <parent link="link_1"/>
       <child link="link_2"/>
-      <limit effort="100000.0" lower="${-pi}" upper="${pi}" velocity="3.14"/>
+      <limit effort="0.0" lower="${-pi}" upper="${pi}" velocity="0.0"/>
       <origin rpy="0 0 0" xyz="${arm_radius} 0 -${arm_len}"/>
+      <!-- <dynamics damping="0.001"/> -->
+      <dynamics friction="0.1"/>
     </joint>
     <transmission name="link_1__link_2_trans">

Commit message: EffortController

File: catkin_ws/src/gibbon/urdf/gibbon.xacro (robot description, xacro)
@@ -61,17 +61,16 @@
       <parent link="link_1"/>
       <child link="link_2"/>
-      <limit effort="0.0" lower="${-pi}" upper="${pi}" velocity="0.0"/>
+      <limit effort="10000.0" lower="${-pi}" upper="${pi}" velocity="0.0"/>
       <origin rpy="0 0 0" xyz="${arm_radius} 0 -${arm_len}"/>
-      <!-- <dynamics damping="0.001"/> -->
-      <dynamics friction="0.1"/>
+      <dynamics friction="0" damping="0.001"/>
     </joint>
     <transmission name="link_1__link_2_trans">
       <type>transmission_interface/SimpleTransmission</type>
       <actuator name="$link_1__link_2_motor">
-        <hardwareInterface>hardware_interface/PositionJointInterface</hardwareInterface>
+        <hardwareInterface>hardware_interface/EffortJointInterface</hardwareInterface>
         <mechanicalReduction>1</mechanicalReduction>
       </actuator>
       <joint name="link_1__link_2">
-        <hardwareInterface>hardware_interface/PositionJointInterface</hardwareInterface>
+        <hardwareInterface>hardware_interface/EffortJointInterface</hardwareInterface>
       </joint>
     </transmission>

Commit message: inertia bugfix

File: catkin_ws/src/gibbon/urdf/gibbon.xacro (robot description, xacro)
@@ -17,5 +17,5 @@
       <inertial>
         <mass value="${mass}" />
-        <inertia ixx="${1.0 / 3.0 * mass * len * len}" ixy="0.0" ixz="0.0" iyy="${1.0 / 3.0 * mass * len * len}" iyz="0.0" izz="0.0" />
+        <inertia ixx="${1.0 / 3.0 * mass * len * len}" ixy="0.0" ixz="0.0" iyy="0" iyz="0.0" izz="0.0" />
       </inertial>
     </xacro:macro>

Commit message: align base link with a gripper

File: catkin_ws/src/gibbon/urdf/gibbon.xacro (robot description, xacro)
@@ -24,5 +24,5 @@
       <parent link="base_link"/>
       <child link="link_1"/>
-      <origin rpy="0 0 0" xyz="0 0 0"/>
+      <origin rpy="0 0 0" xyz="0 0 -0.1"/>
     </joint>
     <link name='link_1'>

Commit message: model velosity limit has chaged

File: catkin_ws/src/gibbon/urdf/gibbon.xacro (robot description, xacro)
@@ -2,5 +2,5 @@
 <robot xmlns:xacro="http://www.ros.org/wiki/xacro" name='gibbon'>
     <xacro:property name="arm_radius" value="0.01" />
-    <xacro:property name="arm_len" value="1" />
+    <xacro:property name="arm_len" value="0.7" />
     <xacro:property name="arm_mass" value="1.0" />
     <xacro:property name="width" value="0.2" />
@@ -61,5 +61,5 @@
       <parent link="link_1"/>
       <child link="link_2"/>
-      <limit effort="10000.0" lower="${-pi}" upper="${pi}" velocity="0.0"/>
+      <limit effort="10000.0" lower="${-pi}" upper="${pi}" velocity="10.0"/>
       <origin rpy="0 0 0" xyz="${arm_radius} 0 -${arm_len}"/>
       <dynamics friction="0" damping="0.001"/>
