Commit message: gibbon xacro: new frame tip && rotate link2 && rm base link

File: catkin_ws/src/gibbon/urdf/gibbon.xacro (robot description, xacro)
@@ -20,10 +20,10 @@
       </inertial>
     </xacro:macro>
-    <link name="base_link"/>
-    <joint name="base_link__link_1" type="fixed">
+    <!-- <link name="base_link"/> -->
+    <!-- <joint name="base_link__link_1" type="fixed">
       <parent link="base_link"/>
       <child link="link_1"/>
       <origin rpy="0 0 0" xyz="0 0 -0.1"/>
-    </joint>
+    </joint> -->
     <link name='link_1'>
       <visual>
@@ -42,7 +42,16 @@
       <xacro:arm_inertial mass="${arm_mass}" len="${arm_len}"/>
     </link>
+    <link name="link_1_tip">
+      <xacro:default_inertial mass="0.00001"/>
+    </link>
+    <joint name="link_1__link_1_tip" type="revolute">
+      <parent link="link_1"/>
+      <child link="link_1_tip"/>
+      <origin rpy="0 0 0" xyz="0 0 0.1"/>
+      <limit lower="0" upper="0" effort="0" velocity="0"/>
+    </joint>
     <link name='link_2'>
       <visual>
-        <origin rpy="0 0 0" xyz="${arm_radius*2} 0 -${arm_len/2}"/>
+        <origin rpy="0 0 0" xyz="${arm_radius*2} 0 ${arm_len/2}"/>
         <material name="grey1"/>
         <geometry>
@@ -51,5 +60,5 @@
       </visual>
       <collision>
-        <origin rpy="0 0 0" xyz="${arm_radius*2} 0 -${arm_len/2}"/>
+        <origin rpy="0 0 0" xyz="${arm_radius*2} 0 ${arm_len/2}"/>
         <geometry>
           <cylinder radius="${arm_radius}" length="${arm_len}"/>
@@ -58,9 +67,18 @@
       <xacro:arm_inertial mass="${arm_mass}" len="${arm_len}"/>
     </link>
+    <link name="link_2_tip">
+      <xacro:default_inertial mass="0.00001"/>
+    </link>
+    <joint name="link_2__link_2_tip" type="revolute">
+      <parent link="link_2"/>
+      <child link="link_2_tip"/>
+      <origin rpy="0 0 0" xyz="${2*arm_radius} 0 ${arm_len + 0.1}"/>
+      <limit lower="0" upper="0" effort="0" velocity="0"/>
+    </joint>
     <joint name="link_1__link_2" type="revolute">
       <parent link="link_1"/>
       <child link="link_2"/>
       <limit effort="10000.0" lower="${-pi}" upper="${pi}" velocity="10.0"/>
-      <origin rpy="0 0 0" xyz="${arm_radius} 0 -${arm_len}"/>
+      <origin rpy="${pi} 0 0" xyz="${arm_radius} 0 -${arm_len}"/>
       <dynamics friction="0" damping="0.001"/>
     </joint>
@@ -83,5 +101,5 @@
       <parent link="link_2"/>
       <child link="link_2_gripper_pole"/>
-      <origin rpy="0 ${pi/2} 0" xyz="${arm_radius*2} 0 -${arm_len}"/>
+      <origin rpy="0 -${pi/2} 0" xyz="${arm_radius*2} 0 ${arm_len}"/>
     </joint>
     <link name="link_1_gripper_pole">
@@ -98,5 +116,5 @@
         <origin xyz="0 0 0" rpy="0 0 0 "/>
       </collision>
-      <xacro:default_inertial mass="0.001"/>
+      <xacro:default_inertial mass="0.00001"/>
     </link>
     <link name="link_2_gripper_pole">
@@ -113,5 +131,5 @@
         <origin xyz="0 0 0" rpy="0 0 0 "/>
       </collision>
-      <xacro:default_inertial mass="0.001"/>
+      <xacro:default_inertial mass="0.00001"/>
     </link>
     <xacro:macro name="gripper" params="prefix reflect link_name">

Commit message: gripper limit 3

File: catkin_ws/src/gibbon/urdf/gibbon.xacro (robot description, xacro)
@@ -136,5 +136,5 @@
       <joint name="${link_name}_${prefix}_gripper_joint" type="revolute">
         <axis xyz="0 0 ${reflect}"/>
-        <limit effort="100000.0" lower="0.0" upper="0.548" velocity="3.14"/>
+        <limit effort="100000.0" lower="0.0" upper="3" velocity="3.14"/>
         <origin rpy="0 0 0" xyz="${polelen} ${reflect*0.01} 0"/>
         <parent link="${link_name}_gripper_pole"/>

Commit message: work with feedback

File: catkin_ws/src/gibbon/urdf/gibbon.xacro (robot description, xacro)
@@ -136,5 +136,5 @@
       <joint name="${link_name}_${prefix}_gripper_joint" type="revolute">
         <axis xyz="0 0 ${reflect}"/>
-        <limit effort="100000.0" lower="0.0" upper="3" velocity="3.14"/>
+        <limit effort="100000.0" lower="0.0" upper="3" velocity="10"/>
         <origin rpy="0 0 0" xyz="${polelen} ${reflect*0.01} 0"/>
         <parent link="${link_name}_gripper_pole"/>

Commit message: inintial state on the ladder

File: catkin_ws/src/gibbon/urdf/gibbon.xacro (robot description, xacro)
@@ -2,5 +2,5 @@
 <robot xmlns:xacro="http://www.ros.org/wiki/xacro" name='gibbon'>
     <xacro:property name="arm_radius" value="0.01" />
-    <xacro:property name="arm_len" value="0.7" />
+    <xacro:property name="arm_len" value="0.8" />
     <xacro:property name="arm_mass" value="1.0" />
     <xacro:property name="width" value="0.2" />
@@ -46,7 +46,7 @@
     </link>
     <joint name="link_1__link_1_tip" type="revolute">
-      <parent link="link_1"/>
-      <child link="link_1_tip"/>
-      <origin rpy="0 0 0" xyz="0 0 0.1"/>
+      <parent link="link_1_tip"/>
+      <child link="link_1"/>
+      <origin rpy="0 0 0" xyz="0 0 -0.1"/>
       <limit lower="0" upper="0" effort="0" velocity="0"/>
     </joint>

Commit message: new urdf props && gripper v shape

File: catkin_ws/src/gibbon/urdf/gibbon.xacro (robot description, xacro)
@@ -1,4 +1,5 @@
 <?xml version='1.0'?>
 <robot xmlns:xacro="http://www.ros.org/wiki/xacro" name='gibbon'>
+    <xacro:include filename="$(find gibbon)/urdf/materials.xacro" />
     <xacro:property name="arm_radius" value="0.01" />
     <xacro:property name="arm_len" value="0.8" />
@@ -45,4 +46,5 @@
       <xacro:default_inertial mass="0.00001"/>
     </link>
+    <!-- <link name="link_1_tip" /> -->
     <joint name="link_1__link_1_tip" type="revolute">
       <parent link="link_1_tip"/>
@@ -79,5 +81,5 @@
       <parent link="link_1"/>
       <child link="link_2"/>
-      <limit effort="10000.0" lower="${-pi}" upper="${pi}" velocity="10.0"/>
+      <limit effort="10000.0" lower="${-pi}" upper="${pi}" velocity="30.0"/>
       <origin rpy="${pi} 0 0" xyz="${arm_radius} 0 -${arm_len}"/>
       <dynamics friction="0" damping="0.001"/>
@@ -159,11 +161,11 @@
         </visual>
         <collision>
+          <origin rpy="${reflect*pi/2} 0 ${reflect*pi/2}" xyz="0.05 0 0"/>
           <geometry>
             <box size="0.001 0.02 0.1"/>
           </geometry>
-          <origin rpy="${reflect*pi/2} 0 ${reflect*pi/2}" xyz="0.05 0 0"/>
         </collision>
         <visual>
-          <origin rpy="0 0 0" xyz="0.1 ${-1*reflect*0.005} 0"/>
+          <origin rpy="0 0.0 ${reflect * 0.7}" xyz="0.104 ${-1*reflect*0.005} 0"/>
           <geometry>
             <box size="0.001 0.01 0.02"/>
@@ -171,8 +173,8 @@
         </visual>
         <collision>
+          <origin rpy="0 0.0 ${reflect * 0.7}" xyz="0.104 ${-1*reflect*0.005} 0"/>
           <geometry>
             <box size="0.001 0.01 0.02"/>
           </geometry>
-          <origin rpy="0 0 0" xyz="0.1 ${-1*reflect*0.005} 0"/>
         </collision>
         <xacro:default_inertial mass="0.05"/>
@@ -183,4 +185,23 @@
     <xacro:gripper prefix="left" reflect="1" link_name="link_2" />
     <xacro:gripper prefix="right" reflect="-1" link_name="link_2" />
+    <gazebo reference="link_1">
+      <material>Gazebo/Red</material>
+    </gazebo>
+    <gazebo reference="link_1_left_gripper">
+      <mu1>1e-00</mu1>
+      <mu2>1e-00</mu2>
+    </gazebo>
+    <gazebo reference="link_1_right_gripper">
+      <mu1>1e-00</mu1>
+      <mu2>1e-00</mu2>
+    </gazebo>
+    <gazebo reference="link_2_left_gripper">
+      <mu1>1e-00</mu1>
+      <mu2>1e-00</mu2>
+    </gazebo>
+    <gazebo reference="link_2_right_gripper">
+      <mu1>1e-00</mu1>
+      <mu2>1e-00</mu2>
+    </gazebo>
     <gazebo>
       <plugin name="gazebo_ros_control" filename="libgazebo_ros_control.so">

File: catkin_ws/src/gibbon/urdf/ladder.xacro (robot description, xacro)
@@ -1,4 +1,5 @@
 <?xml version='1.0'?>
-<robot  name="ladder">
+<robot xmlns:xacro="http://www.ros.org/wiki/xacro" name="ladder">
+  <xacro:include filename="$(find gibbon)/urdf/materials.xacro" />
   <!-- <link name='ladder__base_link'/> -->
   <!-- <joint name="l_b_0" type="revolute">
@@ -194,28 +195,32 @@
     </collision>
   </link>
-    <gazebo reference="ladder__link_0">
-      <mu1>0.001</mu1>
-      <mu2>0.001</mu2>
-      <kp>0.001</kp>
-      <kd>0.001</kd>
-    </gazebo>
-    <gazebo reference="ladder__link_1">
-      <mu1>0.001</mu1>
-      <mu2>0.001</mu2>
-      <kp>0.001</kp>
-      <kd>0.001</kd>
-    </gazebo>
-    <gazebo reference="ladder__link_2">
-      <mu1>0.001</mu1>
-      <mu2>0.001</mu2>
-      <kp>0.001</kp>
-      <kd>0.001</kd>
-    </gazebo>
-    <gazebo reference="ladder__link_3">
-      <mu1>0.001</mu1>
-      <mu2>0.001</mu2>
-      <kp>0.001</kp>
-      <kd>0.001</kd>
-    </gazebo>
+  <gazebo reference="ladder__link_0">
+    <mu1>1</mu1>
+    <mu2>1</mu2>
+    <kp>0</kp>
+    <kd>0</kd>
+    <material>Gazebo/Black</material>
+  </gazebo>
+  <gazebo reference="ladder__link_1">
+    <mu1>1</mu1>
+    <mu2>1</mu2>
+    <kp>0</kp>
+    <kd>0</kd>
+    <material>Gazebo/Black</material>
+  </gazebo>
+  <gazebo reference="ladder__link_2">
+    <mu1>1</mu1>
+    <mu2>1</mu2>
+    <kp>0</kp>
+    <kd>0</kd>
+    <material>Gazebo/Black</material>
+  </gazebo>
+  <gazebo reference="ladder__link_3">
+    <mu1>1</mu1>
+    <mu2>1</mu2>
+    <kp>0</kp>
+    <kd>0</kd>
+    <material>Gazebo/Black</material>
+  </gazebo>
   <gazebo>
     <static>true</static>

Commit message: gibbon inertial rework

File: catkin_ws/src/gibbon/urdf/gibbon.xacro (robot description, xacro)
@@ -18,14 +18,13 @@
       <inertial>
         <mass value="${mass}" />
-        <inertia ixx="${1.0 / 3.0 * mass * len * len}" ixy="0.0" ixz="0.0" iyy="0" iyz="0.0" izz="0.0" />
+        <inertia ixx="${1.0 / 3.0 * mass * len * len}" ixy="0.0" ixz="0.0" iyy="${1.0 / 3.0 * mass * len * len}" iyz="0.0" izz="0.001" />
       </inertial>
     </xacro:macro>
-    <!-- <link name="base_link"/> -->
-    <!-- <joint name="base_link__link_1" type="fixed">
-      <parent link="base_link"/>
-      <child link="link_1"/>
-      <origin rpy="0 0 0" xyz="0 0 -0.1"/>
-    </joint> -->
     <link name='link_1'>
+      <inertial>
+        <mass value="${arm_mass}" />
+        <inertia ixx="0.21" ixy="0.0" ixz="0.0" iyy="0.21" iyz="0.0" izz="0.05" />
+        <origin rpy="0 0 0" xyz="0 0 -${arm_len/2}"/>
+      </inertial>
       <visual>
         <origin rpy="0 0 0" xyz="0 0 -${arm_len/2}"/>
@@ -41,5 +40,4 @@
         </geometry>
       </collision>
-      <xacro:arm_inertial mass="${arm_mass}" len="${arm_len}"/>
     </link>
     <link name="link_1_tip">
@@ -54,6 +52,11 @@
     </joint>
     <link name='link_2'>
-      <visual>
-        <origin rpy="0 0 0" xyz="${arm_radius*2} 0 ${arm_len/2}"/>
+      <inertial>
+        <origin rpy="0 0 0" xyz="0 0 ${arm_len/2}"/>
+        <mass value="${arm_mass}" />
+        <inertia ixx="0.21" ixy="0.0" ixz="0.0" iyy="0.21" iyz="0.0" izz="0.01" />
+      </inertial>
+      <visual>
+        <origin rpy="0 0 0" xyz="0 0 ${arm_len/2}"/>
         <material name="grey1"/>
         <geometry>
@@ -62,10 +65,9 @@
       </visual>
       <collision>
-        <origin rpy="0 0 0" xyz="${arm_radius*2} 0 ${arm_len/2}"/>
-        <geometry>
-          <cylinder radius="${arm_radius}" length="${arm_len}"/>
-        </geometry>
-      </collision>
-      <xacro:arm_inertial mass="${arm_mass}" len="${arm_len}"/>
+        <origin rpy="0 0 0" xyz="0 0 ${arm_len/2}"/>
+        <geometry>
+          <cylinder radius="${arm_radius}" length="${arm_len}"/>
+        </geometry>
+      </collision>
     </link>
     <link name="link_2_tip">
@@ -81,7 +83,7 @@
       <parent link="link_1"/>
       <child link="link_2"/>
-      <limit effort="10000.0" lower="${-pi}" upper="${pi}" velocity="30.0"/>
+      <limit effort="1000.0" lower="${-2*pi}" upper="${2*pi}" velocity="30.0"/>
       <origin rpy="${pi} 0 0" xyz="${arm_radius} 0 -${arm_len}"/>
-      <dynamics friction="0" damping="0.001"/>
+      <dynamics friction="0.0" damping="0.0"/>
     </joint>
     <transmission name="link_1__link_2_trans">
@@ -103,5 +105,5 @@
       <parent link="link_2"/>
       <child link="link_2_gripper_pole"/>
-      <origin rpy="0 -${pi/2} 0" xyz="${arm_radius*2} 0 ${arm_len}"/>
+      <origin rpy="0 -${pi/2} 0" xyz="0 0 ${arm_len}"/>
     </joint>
     <link name="link_1_gripper_pole">
@@ -138,5 +140,5 @@
       <joint name="${link_name}_${prefix}_gripper_joint" type="revolute">
         <axis xyz="0 0 ${reflect}"/>
-        <limit effort="100000.0" lower="0.0" upper="3" velocity="10"/>
+        <limit effort="1000.0" lower="0.0" upper="3" velocity="30"/>
         <origin rpy="0 0 0" xyz="${polelen} ${reflect*0.01} 0"/>
         <parent link="${link_name}_gripper_pole"/>
@@ -189,18 +191,18 @@
     </gazebo>
     <gazebo reference="link_1_left_gripper">
-      <mu1>1e-00</mu1>
-      <mu2>1e-00</mu2>
+      <mu1>1e-01</mu1>
+      <mu2>1e-01</mu2>
     </gazebo>
     <gazebo reference="link_1_right_gripper">
-      <mu1>1e-00</mu1>
-      <mu2>1e-00</mu2>
+      <mu1>1e-01</mu1>
+      <mu2>1e-01</mu2>
     </gazebo>
     <gazebo reference="link_2_left_gripper">
-      <mu1>1e-00</mu1>
-      <mu2>1e-00</mu2>
+      <mu1>1e-01</mu1>
+      <mu2>1e-01</mu2>
     </gazebo>
     <gazebo reference="link_2_right_gripper">
-      <mu1>1e-00</mu1>
-      <mu2>1e-00</mu2>
+      <mu1>1e-01</mu1>
+      <mu2>1e-01</mu2>
     </gazebo>
     <gazebo>
