Commit message: inertia rework

File: catkin_ws/src/gibbon/urdf/gibbon.xacro (robot description, xacro)
@@ -2,92 +2,105 @@
 <robot xmlns:xacro="http://www.ros.org/wiki/xacro" name='gibbon'>
     <xacro:include filename="$(find gibbon)/urdf/materials.xacro" />
+    <xacro:property name="PI" value="3.1415926535897931"/>
     <xacro:property name="arm_radius" value="0.01" />
     <xacro:property name="arm_len" value="0.8" />
     <xacro:property name="arm_mass" value="1.0" />
     <xacro:property name="width" value="0.2" />
-    <xacro:property name="polelen" value="0.0" />
-    <material name="grey1"><color rgba="0.7 0.7 0.7 1"/></material>
-    <material name="grey2"><color rgba="0.9 0.9 0.9 1"/></material>
-    <xacro:macro name="default_inertial" params="mass">
-      <inertial>
-        <mass value="${mass}" />
-        <inertia ixx="1.0" ixy="0.0" ixz="0.0" iyy="1.0" iyz="0.0" izz="1.0" />
-      </inertial>
+    <xacro:property name="polelen" value="0.0001" />
+    <xacro:macro name="box_inertia" params="mass width height">
+      <inertia
+        ixx="${mass / 12.0 * (width*width + height*height)}"
+        ixy="0.0"
+        ixz="0.0"
+        iyy="${mass / 12.0 * (height*height + width*width)}"
+        iyz="0.0"
+        izz="${mass / 12.0 * (width*width + width*width)}"/>
     </xacro:macro>
-    <xacro:macro name="arm_inertial" params="mass len">
-      <inertial>
-        <mass value="${mass}" />
-        <inertia ixx="${1.0 / 3.0 * mass * len * len}" ixy="0.0" ixz="0.0" iyy="${1.0 / 3.0 * mass * len * len}" iyz="0.0" izz="0.001" />
-      </inertial>
-    </xacro:macro>
+    <!-- <link name="world"/>
+    <joint name="fixed" type="fixed">
+      <parent link="world"/>
+      <child link="link_1"/>
+    </joint> -->
     <link name='link_1'>
+      <collision>
+        <origin rpy="0 0 0" xyz="0 0 -${arm_len/2}"/>
+        <geometry>
+          <!-- <cylinder radius="${arm_radius}" length="${arm_len}"/> -->
+          <box size="${arm_radius} ${arm_radius} ${arm_len}"/>
+        </geometry>
+      </collision>
+      <visual>
+        <origin rpy="0 0 0" xyz="0 0 -${arm_len/2}"/>
+        <material name="grey2"/>
+        <geometry>
+          <!-- <cylinder radius="${arm_radius}" length="${arm_len}"/> -->
+          <box size="${arm_radius} ${arm_radius} ${arm_len}"/>
+        </geometry>
+      </visual>
       <inertial>
         <mass value="${arm_mass}" />
-        <inertia ixx="0.21" ixy="0.0" ixz="0.0" iyy="0.21" iyz="0.0" izz="0.05" />
-        <origin rpy="0 0 0" xyz="0 0 -${arm_len/2}"/>
-      </inertial>
-      <visual>
-        <origin rpy="0 0 0" xyz="0 0 -${arm_len/2}"/>
-        <material name="grey2"/>
-        <geometry>
-          <cylinder radius="${arm_radius}" length="${arm_len}"/>
-        </geometry>
-      </visual>
-      <collision>
-        <origin rpy="0 0 0" xyz="0 0 -${arm_len/2}"/>
-        <geometry>
-          <cylinder radius="${arm_radius}" length="${arm_len}"/>
-        </geometry>
-      </collision>
-    </link>
-    <link name="link_1_tip">
-      <xacro:default_inertial mass="0.00001"/>
-    </link>
+        <origin rpy="0 0 0" xyz="0 0 -${arm_len/2}"/>
+        <xacro:box_inertia mass="${arm_mass}" width="${arm_radius}" height="${arm_len}" />
+      </inertial>
+    </link>
+    <!-- <link name="link_1_tip">
+      <inertial>
+        <mass value="0.001" />
+        <origin rpy="0 0 0" xyz="0 0 0"/>
+        <xacro:box_inertia mass="0.001" width="0.001" height="0.001" />
+      </inertial>
+    </link> -->
     <!-- <link name="link_1_tip" /> -->
-    <joint name="link_1__link_1_tip" type="revolute">
+    <!-- <joint name="link_1__link_1_tip" type="revolute">
       <parent link="link_1_tip"/>
       <child link="link_1"/>
       <origin rpy="0 0 0" xyz="0 0 -0.1"/>
       <limit lower="0" upper="0" effort="0" velocity="0"/>
-    </joint>
+    </joint> -->
     <link name='link_2'>
+      <collision>
+        <origin rpy="0 0 0" xyz="0 0 ${arm_len/2}"/>
+        <geometry>
+          <!-- <cylinder radius="${arm_radius}" length="${arm_len}"/> -->
+          <box size="${arm_radius} ${arm_radius} ${arm_len}"/>
+        </geometry>
+      </collision>
+      <visual>
+        <origin rpy="0 0 0" xyz="0 0 ${arm_len/2}"/>
+        <material name="grey1"/>
+        <geometry>
+          <!-- <cylinder radius="${arm_radius}" length="${arm_len}"/> -->
+          <box size="${arm_radius} ${arm_radius} ${arm_len}"/>
+        </geometry>
+      </visual>
       <inertial>
         <origin rpy="0 0 0" xyz="0 0 ${arm_len/2}"/>
         <mass value="${arm_mass}" />
-        <inertia ixx="0.21" ixy="0.0" ixz="0.0" iyy="0.21" iyz="0.0" izz="0.01" />
-      </inertial>
-      <visual>
-        <origin rpy="0 0 0" xyz="0 0 ${arm_len/2}"/>
-        <material name="grey1"/>
-        <geometry>
-          <cylinder radius="${arm_radius}" length="${arm_len}"/>
-        </geometry>
-      </visual>
-      <collision>
-        <origin rpy="0 0 0" xyz="0 0 ${arm_len/2}"/>
-        <geometry>
-          <cylinder radius="${arm_radius}" length="${arm_len}"/>
-        </geometry>
-      </collision>
-    </link>
-    <link name="link_2_tip">
-      <xacro:default_inertial mass="0.00001"/>
-    </link>
-    <joint name="link_2__link_2_tip" type="revolute">
+        <xacro:box_inertia mass="${arm_mass}" width="${arm_radius}" height="${arm_len}" />
+      </inertial>
+    </link>
+    <!-- <link name="link_2_tip">
+      <inertial>
+        <mass value="${arm_mass}" />
+        <origin rpy="0 0 0" xyz="0 0 -${arm_len/2}"/>
+        <xacro:box_inertia mass="${arm_mass}" width="${arm_radius}" height="${arm_len}" />
+      </inertial>
+    </link> -->
+    <!-- <joint name="link_2__link_2_tip" type="revolute">
       <parent link="link_2"/>
       <child link="link_2_tip"/>
       <origin rpy="0 0 0" xyz="${2*arm_radius} 0 ${arm_len + 0.1}"/>
       <limit lower="0" upper="0" effort="0" velocity="0"/>
-    </joint>
-    <joint name="link_1__link_2" type="revolute">
+    </joint> -->
+    <joint name="link_1__link_2" type="continuous">
       <parent link="link_1"/>
       <child link="link_2"/>
-      <limit effort="1000.0" lower="${-2*pi}" upper="${2*pi}" velocity="30.0"/>
-      <origin rpy="${pi} 0 0" xyz="${arm_radius} 0 -${arm_len}"/>
-      <dynamics friction="0.0" damping="0.0"/>
+      <!-- <limit effort="1000.0" lower="${-2*PI}" upper="${2*PI}" velocity="30.0"/> -->
+      <origin rpy="${PI} 0 0" xyz="${2 * arm_radius + 0.001} 0 -${arm_len}"/>
+      <dynamics friction="0.0" damping="0.01"/>
     </joint>
     <transmission name="link_1__link_2_trans">
       <type>transmission_interface/SimpleTransmission</type>
-      <actuator name="$link_1__link_2_motor">
+      <actuator name="link_1__link_2_motor">
         <hardwareInterface>hardware_interface/EffortJointInterface</hardwareInterface>
         <mechanicalReduction>1</mechanicalReduction>
@@ -100,17 +113,36 @@
       <parent link="link_1"/>
       <child link="link_1_gripper_pole"/>
-      <origin rpy="0 -${pi/2} 0" xyz="0 0 0"/>
+      <origin rpy="0 -${PI/2} 0" xyz="0 0 0"/>
     </joint>
     <joint name="link_2__gripper" type="fixed">
       <parent link="link_2"/>
       <child link="link_2_gripper_pole"/>
-      <origin rpy="0 -${pi/2} 0" xyz="0 0 ${arm_len}"/>
+      <origin rpy="0 -${PI/2} 0" xyz="0 0 ${arm_len}"/>
     </joint>
     <link name="link_1_gripper_pole">
       <visual>
         <geometry>
+          <cylinder length="${polelen}" radius="${polelen}"/>
+        </geometry>
+        <origin xyz="0 0 0" rpy="0 0 0 "/>
+      </visual>
+      <collision>
+        <geometry>
           <cylinder length="${polelen}" radius="0.01"/>
         </geometry>
         <origin xyz="0 0 0" rpy="0 0 0 "/>
+      </collision>
+      <inertial>
+        <mass value="${polelen}" />
+        <origin xyz="0 0 0" rpy="0 0 0 "/>
+        <xacro:box_inertia mass="${polelen}" width="${polelen}" height="${polelen}" />
+      </inertial>
+    </link>
+    <link name="link_2_gripper_pole">
+      <visual>
+        <geometry>
+          <cylinder length="${polelen}" radius="${polelen}"/>
+        </geometry>
+        <origin xyz="0 0 0" rpy="0 0 0 "/>
       </visual>
       <collision>
@@ -120,20 +152,9 @@
         <origin xyz="0 0 0" rpy="0 0 0 "/>
       </collision>
-      <xacro:default_inertial mass="0.00001"/>
-    </link>
-    <link name="link_2_gripper_pole">
-      <visual>
-        <geometry>
-          <cylinder length="${polelen}" radius="0.01"/>
-        </geometry>
-        <origin xyz="0 0 0" rpy="0 0 0 "/>
-      </visual>
-      <collision>
-        <geometry>
-          <cylinder length="${polelen}" radius="0.01"/>
-        </geometry>
-        <origin xyz="0 0 0" rpy="0 0 0 "/>
-      </collision>
-      <xacro:default_inertial mass="0.00001"/>
+      <inertial>
+        <mass value="${polelen}" />
+        <origin xyz="0 0 0" rpy="0 0 0 "/>
+        <xacro:box_inertia mass="${polelen}" width="${polelen}" height="${polelen}" />
+      </inertial>
     </link>
     <xacro:macro name="gripper" params="prefix reflect link_name">
@@ -157,5 +178,5 @@
       <link name="${link_name}_${prefix}_gripper">
         <visual>
-          <origin rpy="${reflect*pi/2} 0 ${reflect*pi/2}" xyz="0.05 0 0"/>
+          <origin rpy="${reflect*PI/2} 0 ${reflect*PI/2}" xyz="0.05 0 0"/>
           <geometry>
             <box size="0.001 0.02 0.1"/>
@@ -163,5 +184,5 @@
         </visual>
         <collision>
-          <origin rpy="${reflect*pi/2} 0 ${reflect*pi/2}" xyz="0.05 0 0"/>
+          <origin rpy="${reflect*PI/2} 0 ${reflect*PI/2}" xyz="0.05 0 0"/>
           <geometry>
             <box size="0.001 0.02 0.1"/>
@@ -180,5 +201,9 @@
           </geometry>
         </collision>
-        <xacro:default_inertial mass="0.05"/>
+        <inertial>
+          <mass value="0.1" />
+          <origin rpy="0 0 0" xyz="0 0.0 0"/>
+          <xacro:box_inertia mass="0.1" width="0.1" height="0.1" />
+        </inertial>
       </link>
     </xacro:macro>
@@ -189,24 +214,39 @@
     <gazebo reference="link_1">
       <material>Gazebo/Red</material>
-    </gazebo>
-    <gazebo reference="link_1_left_gripper">
-      <mu1>1e-01</mu1>
-      <mu2>1e-01</mu2>
+      <mu1>1e-01</mu1>
+      <mu2>1e-01</mu2>
+    </gazebo>
+    <gazebo reference="link_2">
+      <mu1>1e-01</mu1>
+      <mu2>1e-01</mu2>
+    </gazebo>
+    <!-- <gazebo reference="link_1_left_gripper">
+      <mu1>1e-01</mu1>
+      <mu2>1e-01</mu2>
+      <kp>0</kp>
+      <kd>0</kd>
     </gazebo>
     <gazebo reference="link_1_right_gripper">
       <mu1>1e-01</mu1>
       <mu2>1e-01</mu2>
+      <kp>0</kp>
+      <kd>0</kd>
     </gazebo>
     <gazebo reference="link_2_left_gripper">
       <mu1>1e-01</mu1>
       <mu2>1e-01</mu2>
+      <kp>0</kp>
+      <kd>0</kd>
     </gazebo>
     <gazebo reference="link_2_right_gripper">
       <mu1>1e-01</mu1>
       <mu2>1e-01</mu2>
-    </gazebo>
+      <kp>0</kp>
+      <kd>0</kd>
+    </gazebo> -->
     <gazebo>
       <plugin name="gazebo_ros_control" filename="libgazebo_ros_control.so">
         <robotNamespace>/gibbon</robotNamespace>
+        <robotSimType>gazebo_ros_control/DefaultRobotHWSim</robotSimType>
       </plugin>
     </gazebo>

File: catkin_ws/src/gibbon/urdf/ladder.xacro (robot description, xacro)
@@ -2,5 +2,9 @@
 <robot xmlns:xacro="http://www.ros.org/wiki/xacro" name="ladder">
   <xacro:include filename="$(find gibbon)/urdf/materials.xacro" />
-  <!-- <link name='ladder__base_link'/> -->
+  <!-- <link name="world"/>
+  <joint name="fixed" type="fixed">
+    <parent link="world"/>
+    <child link="ladder__link_0"/>
+  </joint> -->
   <!-- <joint name="l_b_0" type="revolute">
     <parent link="ladder__base_link"/>
@@ -29,4 +33,5 @@
   <link name='ladder__link_0'>
     <inertial>
+      <origin rpy="1.57 0 0" xyz="0 0.15 3"/>
       <mass value="1.0"/>
       <inertia ixx="0.1633333333333333" ixy="0.0" ixz="0.0" iyy="0" iyz="0.0" izz="0.0"/>
@@ -71,4 +76,5 @@
   <link name='ladder__link_1'>
     <inertial>
+      <origin rpy="1.57 0 0" xyz="1.4 0.15 3"/>
       <mass value="1.0"/>
       <inertia ixx="0.1633333333333333" ixy="0.0" ixz="0.0" iyy="0" iyz="0.0" izz="0.0"/>
@@ -113,4 +119,5 @@
   <link name='ladder__link_2'>
     <inertial>
+      <origin rpy="1.57 0 0" xyz="2.8 0.15 3"/>
       <mass value="1.0"/>
       <inertia ixx="0.1633333333333333" ixy="0.0" ixz="0.0" iyy="0" iyz="0.0" izz="0.0"/>
@@ -155,4 +162,5 @@
   <link name='ladder__link_3'>
     <inertial>
+      <origin rpy="1.57 0 0" xyz="4.2 0.15 3"/>
       <mass value="1.0"/>
       <inertia ixx="0.1633333333333333" ixy="0.0" ixz="0.0" iyy="0" iyz="0.0" izz="0.0"/>
@@ -195,5 +203,5 @@
     </collision>
   </link>
-  <gazebo reference="ladder__link_0">
+  <!-- <gazebo reference="ladder__link_0">
     <mu1>1e-03</mu1>
     <mu2>1e-03</mu2>
@@ -222,5 +230,5 @@
     <kd>0</kd>
     <material>Gazebo/Black</material>
-  </gazebo>
+  </gazebo> -->
   <gazebo>
     <static>true</static>

Commit message: gibbon tip added

File: catkin_ws/src/gibbon/urdf/gibbon.xacro (robot description, xacro)
@@ -44,5 +44,5 @@
       </inertial>
     </link>
-    <!-- <link name="link_1_tip">
+    <link name="link_1_tip">
       <inertial>
         <mass value="0.001" />
@@ -50,12 +50,12 @@
         <xacro:box_inertia mass="0.001" width="0.001" height="0.001" />
       </inertial>
-    </link> -->
+    </link>
     <!-- <link name="link_1_tip" /> -->
-    <!-- <joint name="link_1__link_1_tip" type="revolute">
+    <joint name="link_1__link_1_tip" type="revolute">
       <parent link="link_1_tip"/>
       <child link="link_1"/>
       <origin rpy="0 0 0" xyz="0 0 -0.1"/>
       <limit lower="0" upper="0" effort="0" velocity="0"/>
-    </joint> -->
+    </joint>
     <link name='link_2'>
       <collision>
@@ -80,5 +80,5 @@
       </inertial>
     </link>
-    <!-- <link name="link_2_tip">
+    <link name="link_2_tip">
       <inertial>
         <mass value="${arm_mass}" />
@@ -86,11 +86,11 @@
         <xacro:box_inertia mass="${arm_mass}" width="${arm_radius}" height="${arm_len}" />
       </inertial>
-    </link> -->
-    <!-- <joint name="link_2__link_2_tip" type="revolute">
+    </link>
+    <joint name="link_2__link_2_tip" type="revolute">
       <parent link="link_2"/>
       <child link="link_2_tip"/>
       <origin rpy="0 0 0" xyz="${2*arm_radius} 0 ${arm_len + 0.1}"/>
       <limit lower="0" upper="0" effort="0" velocity="0"/>
-    </joint> -->
+    </joint>
     <joint name="link_1__link_2" type="continuous">
       <parent link="link_1"/>
@@ -98,5 +98,5 @@
       <!-- <limit effort="1000.0" lower="${-2*PI}" upper="${2*PI}" velocity="30.0"/> -->
       <origin rpy="${PI} 0 0" xyz="${2 * arm_radius + 0.001} 0 -${arm_len}"/>
-      <dynamics friction="0.0" damping="0.01"/>
+      <dynamics friction="0.0" damping="0.0"/>
     </joint>
     <transmission name="link_1__link_2_trans">
@@ -168,5 +168,5 @@
       <transmission name="${link_name}_${prefix}_gripper_joint_trans">
         <type>transmission_interface/SimpleTransmission</type>
-        <actuator name="$${link_name}_${prefix}_gripper_joint_motor">
+        <actuator name="${link_name}_${prefix}_gripper_joint_motor">
           <hardwareInterface>hardware_interface/PositionJointInterface</hardwareInterface>
           <mechanicalReduction>1</mechanicalReduction>
@@ -203,5 +203,5 @@
         <inertial>
           <mass value="0.1" />
-          <origin rpy="0 0 0" xyz="0 0.0 0"/>
+          <origin rpy="0 0 0" xyz="0 0 0"/>
           <xacro:box_inertia mass="0.1" width="0.1" height="0.1" />
         </inertial>

Commit message: no tip

File: catkin_ws/src/gibbon/urdf/gibbon.xacro (robot description, xacro)
@@ -44,18 +44,18 @@
       </inertial>
     </link>
-    <link name="link_1_tip">
-      <inertial>
-        <mass value="0.001" />
+    <!-- <link name="link_1_tip">
+      <inertial>
+        <mass value="0.0001" />
         <origin rpy="0 0 0" xyz="0 0 0"/>
-        <xacro:box_inertia mass="0.001" width="0.001" height="0.001" />
-      </inertial>
-    </link>
+        <xacro:box_inertia mass="0.0001" width="0.0001" height="0.0001" />
+      </inertial>
+    </link> -->
     <!-- <link name="link_1_tip" /> -->
-    <joint name="link_1__link_1_tip" type="revolute">
+    <!-- <joint name="link_1__link_1_tip" type="revolute">
       <parent link="link_1_tip"/>
       <child link="link_1"/>
       <origin rpy="0 0 0" xyz="0 0 -0.1"/>
       <limit lower="0" upper="0" effort="0" velocity="0"/>
-    </joint>
+    </joint> -->
     <link name='link_2'>
       <collision>
@@ -80,17 +80,17 @@
       </inertial>
     </link>
-    <link name="link_2_tip">
-      <inertial>
-        <mass value="${arm_mass}" />
-        <origin rpy="0 0 0" xyz="0 0 -${arm_len/2}"/>
-        <xacro:box_inertia mass="${arm_mass}" width="${arm_radius}" height="${arm_len}" />
-      </inertial>
-    </link>
-    <joint name="link_2__link_2_tip" type="revolute">
+    <!-- <link name="link_2_tip">
+      <inertial>
+        <mass value="0.0001" />
+        <origin rpy="0 0 0" xyz="0 0 -${arm_len/2}"/>
+        <xacro:box_inertia mass="0.0001" width="0.0001" height="0.0001" />
+      </inertial>
+    </link> -->
+    <!-- <joint name="link_2__link_2_tip" type="revolute">
       <parent link="link_2"/>
       <child link="link_2_tip"/>
       <origin rpy="0 0 0" xyz="${2*arm_radius} 0 ${arm_len + 0.1}"/>
       <limit lower="0" upper="0" effort="0" velocity="0"/>
-    </joint>
+    </joint> -->
     <joint name="link_1__link_2" type="continuous">
       <parent link="link_1"/>
@@ -159,19 +159,22 @@
     </link>
     <xacro:macro name="gripper" params="prefix reflect link_name">
-      <joint name="${link_name}_${prefix}_gripper_joint" type="revolute">
+      <joint name="${link_name}_${prefix}_gripper_joint" type="continuous">
         <axis xyz="0 0 ${reflect}"/>
-        <limit effort="1000.0" lower="0.0" upper="3" velocity="30"/>
-        <origin rpy="0 0 0" xyz="${polelen} ${reflect*0.01} 0"/>
+        <!-- <limit effort="1000.0" lower="0.0" upper="3" velocity="30"/> -->
+        <origin rpy="0 0 0" xyz="${polelen} ${reflect*0.012} 0"/>
         <parent link="${link_name}_gripper_pole"/>
         <child link="${link_name}_${prefix}_gripper"/>
+        <dynamics friction="0.0" damping="0.0"/>
       </joint>
       <transmission name="${link_name}_${prefix}_gripper_joint_trans">
         <type>transmission_interface/SimpleTransmission</type>
         <actuator name="${link_name}_${prefix}_gripper_joint_motor">
-          <hardwareInterface>hardware_interface/PositionJointInterface</hardwareInterface>
+          <hardwareInterface>hardware_interface/EffortJointInterface</hardwareInterface>
+          <!-- <hardwareInterface>hardware_interface/PositionJointInterface</hardwareInterface> -->
           <mechanicalReduction>1</mechanicalReduction>
         </actuator>
         <joint name="${link_name}_${prefix}_gripper_joint">
-          <hardwareInterface>hardware_interface/PositionJointInterface</hardwareInterface>
+          <hardwareInterface>hardware_interface/EffortJointInterface</hardwareInterface>
+          <!-- <hardwareInterface>hardware_interface/PositionJointInterface</hardwareInterface> -->
         </joint>
       </transmission>
@@ -192,5 +195,5 @@
           <origin rpy="0 0.0 ${reflect * 0.7}" xyz="0.104 ${-1*reflect*0.005} 0"/>
           <geometry>
-            <box size="0.001 0.01 0.02"/>
+            <box size="0.001 0.02 0.02"/>
           </geometry>
         </visual>
@@ -198,5 +201,5 @@
           <origin rpy="0 0.0 ${reflect * 0.7}" xyz="0.104 ${-1*reflect*0.005} 0"/>
           <geometry>
-            <box size="0.001 0.01 0.02"/>
+            <box size="0.001 0.02 0.02"/>
           </geometry>
         </collision>

Commit message: gripper with limits

File: catkin_ws/src/gibbon/urdf/gibbon.xacro (robot description, xacro)
@@ -159,8 +159,8 @@
     </link>
     <xacro:macro name="gripper" params="prefix reflect link_name">
-      <joint name="${link_name}_${prefix}_gripper_joint" type="continuous">
+      <joint name="${link_name}_${prefix}_gripper_joint" type="revolute">
         <axis xyz="0 0 ${reflect}"/>
-        <!-- <limit effort="1000.0" lower="0.0" upper="3" velocity="30"/> -->
-        <origin rpy="0 0 0" xyz="${polelen} ${reflect*0.012} 0"/>
+        <limit effort="100.0" lower="0.0" upper="3" velocity="10"/>
+        <origin rpy="0 0 0" xyz="${polelen} ${reflect*0.014} 0"/>
         <parent link="${link_name}_gripper_pole"/>
         <child link="${link_name}_${prefix}_gripper"/>
